Commit message: add wbc control for h1
Signed-off-by: djh <djh199512@163.com>

File: resources/robot/h1/urdf/h1.urdf (robot description, URDF)
Before this commit: robot h1_description, 22 links, 21 joints
Links:
- removed link imu_link
- removed link left_ankle_link
- removed link left_elbow_link
- removed link left_hip_pitch_link
- removed link left_hip_roll_link
- removed link left_hip_yaw_link
- removed link left_knee_link
- removed link left_shoulder_pitch_link
- removed link left_shoulder_roll_link
- removed link left_shoulder_yaw_link
- removed link logo_link
- removed link pelvis
- removed link right_ankle_link
- removed link right_elbow_link
- removed link right_hip_pitch_link
- removed link right_hip_roll_link
- removed link right_hip_yaw_link
- removed link right_knee_link
- removed link right_shoulder_pitch_link
- removed link right_shoulder_roll_link
- removed link right_shoulder_yaw_link
- removed link torso_link
- added link Link_ankle_l_pitch, mass 0.10145; collision mesh filename=package://AzureLoong/meshes/Link_ankle_l_pitch.STL; visual mesh filename=package://AzureLoong/meshes/Link_ankle_l_pitch.STL
- added link Link_ankle_l_roll, mass 0.7522882; collision mesh filename=package://AzureLoong/meshes/Link_ankle_l_roll.STL; visual mesh filename=package://AzureLoong/meshes/Link_ankle_l_roll.STL
- added link Link_ankle_r_pitch, mass 0.10145; collision mesh filename=package://AzureLoong/meshes/Link_ankle_r_pitch.STL; visual mesh filename=package://AzureLoong/meshes/Link_ankle_r_pitch.STL
- added link Link_ankle_r_roll, mass 0.75229; collision mesh filename=package://AzureLoong/meshes/Link_ankle_r_roll.STL; visual mesh filename=package://AzureLoong/meshes/Link_ankle_r_roll.STL
- added link Link_arm_l_01, mass 0.756406339732892; collision mesh filename=package://AzureLoong/meshes/Link_arm_l_01.STL; visual mesh filename=package://AzureLoong/meshes/Link_arm_l_01.STL
- added link Link_arm_l_02, mass 0.984999996273518; collision mesh filename=package://AzureLoong/meshes/Link_arm_l_02.STL; visual mesh filename=package://AzureLoong/meshes/Link_arm_l_02.STL
- added link Link_arm_l_03, mass 0.958999855228925; collision mesh filename=package://AzureLoong/meshes/Link_arm_l_03.STL; visual mesh filename=package://AzureLoong/meshes/Link_arm_l_03.STL
- added link Link_arm_l_04, mass 0.60000012303258; collision mesh filename=package://AzureLoong/meshes/Link_arm_l_04.STL; visual mesh filename=package://AzureLoong/meshes/Link_arm_l_04.STL
- added link Link_arm_l_05, mass 0.68976; collision mesh filename=package://AzureLoong/meshes/Link_arm_l_05.STL; visual mesh filename=package://AzureLoong/meshes/Link_arm_l_05.STL
- added link Link_arm_l_06, mass 0.280000012776158; collision mesh filename=package://AzureLoong/meshes/Link_arm_l_06.STL; visual mesh filename=package://AzureLoong/meshes/Link_arm_l_06.STL
- added link Link_arm_l_07, mass 0.61354; collision mesh filename=package://AzureLoong/meshes/Link_arm_l_07.STL; visual mesh filename=package://AzureLoong/meshes/Link_arm_l_07.STL
- added link Link_arm_r_01, mass 0.75641; collision mesh filename=package://AzureLoong/meshes/Link_arm_r_01.STL; visual mesh filename=package://AzureLoong/meshes/Link_arm_r_01.STL
- added link Link_arm_r_02, mass 0.984999996273518; collision mesh filename=package://AzureLoong/meshes/Link_arm_r_02.STL; visual mesh filename=package://AzureLoong/meshes/Link_arm_r_02.STL
- added link Link_arm_r_03, mass 0.958999855228924; collision mesh filename=package://AzureLoong/meshes/Link_arm_r_03.STL; visual mesh filename=package://AzureLoong/meshes/Link_arm_r_03.STL
- added link Link_arm_r_04, mass 0.6; collision mesh filename=package://AzureLoong/meshes/Link_arm_r_04.STL; visual mesh filename=package://AzureLoong/meshes/Link_arm_r_04.STL
- added link Link_arm_r_05, mass 0.68976; collision mesh filename=package://AzureLoong/meshes/Link_arm_r_05.STL; visual mesh filename=package://AzureLoong/meshes/Link_arm_r_05.STL
- added link Link_arm_r_06, mass 0.28; collision mesh filename=package://AzureLoong/meshes/Link_arm_r_06.STL; visual mesh filename=package://AzureLoong/meshes/Link_arm_r_06.STL
- added link Link_arm_r_07, mass 0.61354; collision mesh filename=package://AzureLoong/meshes/Link_arm_r_07.STL; visual mesh filename=package://AzureLoong/meshes/Link_arm_r_07.STL
- added link Link_head_pitch, mass 1.3943; collision mesh filename=package://AzureDragon/meshes/Link_head_pitch.STL; visual mesh filename=package://AzureDragon/meshes/Link_head_pitch.STL
- added link Link_head_yaw, mass 0.84249; collision mesh filename=package://AzureDragon/meshes/Link_head_yaw.STL; visual mesh filename=package://AzureDragon/meshes/Link_head_yaw.STL
- added link Link_hip_l_pitch, mass 5.2378; collision mesh filename=package://AzureLoong/meshes/Link_hip_l_pitch.STL; visual mesh filename=package://AzureLoong/meshes/Link_hip_l_pitch.STL
- added link Link_hip_l_roll, mass 2.4334; collision mesh filename=package://AzureLoong/meshes/Link_hip_l_roll.STL; visual mesh filename=package://AzureLoong/meshes/Link_hip_l_roll.STL
- added link Link_hip_l_yaw, mass 3.4304; collision mesh filename=package://AzureLoong/meshes/Link_hip_l_yaw.STL; visual mesh filename=package://AzureLoong/meshes/Link_hip_l_yaw.STL
- added link Link_hip_r_pitch, mass 5.2378; collision mesh filename=package://AzureLoong/meshes/Link_hip_r_pitch.STL; visual mesh filename=package://AzureLoong/meshes/Link_hip_r_pitch.STL
- added link Link_hip_r_roll, mass 2.4334; collision mesh filename=package://AzureLoong/meshes/Link_hip_r_roll.STL; visual mesh filename=package://AzureLoong/meshes/Link_hip_r_roll.STL
- added link Link_hip_r_yaw, mass 3.4303; collision mesh filename=package://AzureLoong/meshes/Link_hip_r_yaw.STL; visual mesh filename=package://AzureLoong/meshes/Link_hip_r_yaw.STL
- added link Link_knee_l_pitch, mass 2.9775; collision mesh filename=package://AzureLoong/meshes/Link_knee_l_pitch.STL; visual mesh filename=package://AzureLoong/meshes/Link_knee_l_pitch.STL
- added link Link_knee_r_pitch, mass 2.9775; collision mesh filename=package://AzureLoong/meshes/Link_knee_r_pitch.STL; visual mesh filename=package://AzureLoong/meshes/Link_knee_r_pitch.STL
- added link Link_waist_pitch, mass 2.6964; collision mesh filename=package://AzureLoong/meshes/Link_waist_pitch.STL; visual mesh filename=package://AzureLoong/meshes/Link_waist_pitch.STL
- added link Link_waist_roll, mass 2.9806; collision mesh filename=package://AzureLoong/meshes/Link_waist_roll.STL; visual mesh filename=package://AzureLoong/meshes/Link_waist_roll.STL
- added link Link_waist_yaw, mass 7.3588; collision mesh filename=package://AzureLoong/meshes/Link_waist_yaw.STL; visual mesh filename=package://AzureLoong/meshes/Link_waist_yaw.STL
- added link base_link, mass 22.447; collision mesh filename=package://AzureLoong/meshes/base_link.STL; visual mesh filename=package://AzureLoong/meshes/base_link.STL
Joints:
- removed joint imu_joint
- removed joint left_ankle_joint
- removed joint left_elbow_joint
- removed joint left_hip_pitch_joint
- removed joint left_hip_roll_joint
- removed joint left_hip_yaw_joint
- removed joint left_knee_joint
- removed joint left_shoulder_pitch_joint
- removed joint left_shoulder_roll_joint
- removed joint left_shoulder_yaw_joint
- removed joint logo_joint
- removed joint right_ankle_joint
- removed joint right_elbow_joint
- removed joint right_hip_pitch_joint
- removed joint right_hip_roll_joint
- removed joint right_hip_yaw_joint
- removed joint right_knee_joint
- removed joint right_shoulder_pitch_joint
- removed joint right_shoulder_roll_joint
- removed joint right_shoulder_yaw_joint
- removed joint torso_joint
- added joint J_ankle_l_pitch: type revolute, parent Link_knee_l_pitch, child Link_ankle_l_pitch, origin xyz=0 0 -0.387 rpy=0 0 0, axis 0 -1 0, limit lower=-0.47 upper=0.87 effort=58.5 velocity=48.8
- added joint J_ankle_l_roll: type revolute, parent Link_ankle_l_pitch, child Link_ankle_l_roll, origin xyz=0 0 0 rpy=0 0 0, axis 1 0 0, limit lower=-0.43633 upper=0.43633 effort=58.5 velocity=48.8
- added joint J_ankle_r_pitch: type revolute, parent Link_knee_r_pitch, child Link_ankle_r_pitch, origin xyz=0 0 -0.387 rpy=0 0 0, axis 0 -1 0, limit lower=-0.47 upper=0.87 effort=58.5 velocity=48.8
- added joint J_ankle_r_roll: type revolute, parent Link_ankle_r_pitch, child Link_ankle_r_roll, origin xyz=0 0 0 rpy=0 0 0, axis 1 0 0, limit lower=-0.43633 upper=0.43633 effort=58.5 velocity=48.8
- added joint J_arm_l_01: type revolute, parent base_link, child Link_arm_l_01, origin xyz=0.004 0.1616 0.3922 rpy=0 0 0, axis 0 1 0, limit lower=-2.96706 upper=2.96706 effort=80 velocity=3.14
- added joint J_arm_l_02: type revolute, parent Link_arm_l_01, child Link_arm_l_02, origin xyz=0.042 0.041 0 rpy=0 0 0, axis 1 0 0, limit lower=-1.83260 upper=1.83260 effort=80 velocity=3.14
- added joint J_arm_l_03: type revolute, parent Link_arm_l_02, child Link_arm_l_03, origin xyz=-0.042 0.1226 0 rpy=0 0 0, axis 0 1 0, limit lower=-2.96706 upper=2.96706 effort=48 velocity=3.14
- added joint J_arm_l_04: type revolute, parent Link_arm_l_03, child Link_arm_l_04, origin xyz=-0.0353 0.1774 0.024 rpy=0 0 0, axis 1 0 0, limit lower=0 upper=2.96706 effort=48 velocity=3.14
- added joint J_arm_l_05: type revolute, parent Link_arm_l_04, child Link_arm_l_05, origin xyz=0.0353 0.1035 -0.024 rpy=0 0 0, axis 0 1 0, limit lower=-2.96706 upper=2.96706 effort=12.4 velocity=6.28
- added joint J_arm_l_06: type revolute, parent Link_arm_l_05, child Link_arm_l_06, origin xyz=0.0265 0.1965 0 rpy=0 0 0, axis -1 0 0, limit lower=-1.8326 upper=1.8326 effort=12.4 velocity=6.28
- added joint J_arm_l_07: type revolute, parent Link_arm_l_06, child Link_arm_l_07, origin xyz=-0.0265 0 0.0318 rpy=0 0 0, axis 0 0 1, limit lower=-1.04720 upper=1.04720 effort=12.4 velocity=6.28
- added joint J_arm_r_01: type revolute, parent base_link, child Link_arm_r_01, origin xyz=0.004 -0.1616 0.3922 rpy=0 0 0, axis 0 -1 0, limit lower=-2.96706 upper=2.96706 effort=80 velocity=3.14
- added joint J_arm_r_02: type revolute, parent Link_arm_r_01, child Link_arm_r_02, origin xyz=-0.042 -0.041 0 rpy=0 0 0, axis -1 0 0, limit lower=-1.83260 upper=1.83260 effort=80 velocity=3.14
- added joint J_arm_r_03: type revolute, parent Link_arm_r_02, child Link_arm_r_03, origin xyz=0.042 -0.1226 0 rpy=0 0 0, axis 0 -1 0, limit lower=-2.96706 upper=2.96706 effort=48 velocity=3.14
- added joint J_arm_r_04: type revolute, parent Link_arm_r_03, child Link_arm_r_04, origin xyz=0.0353 -0.1774 0.024 rpy=0 0 0, axis -1 0 0, limit lower=0 upper=2.96706 effort=48 velocity=3.14
- added joint J_arm_r_05: type revolute, parent Link_arm_r_04, child Link_arm_r_05, origin xyz=-0.0353 -0.1035 -0.024 rpy=0 0 0, axis 0 -1 0, limit lower=-2.96706 upper=2.96706 effort=12.4 velocity=6.28
- added joint J_arm_r_06: type revolute, parent Link_arm_r_05, child Link_arm_r_06, origin xyz=-0.0265 -0.1965 0 rpy=0 0 0, axis 1 0 0, limit lower=-1.8326 upper=1.8326 effort=12.4 velocity=6.28
- added joint J_arm_r_07: type revolute, parent Link_arm_r_06, child Link_arm_r_07, origin xyz=0.0265 0 0.0318 rpy=0 0 0, axis 0 0 1, limit lower=-1.04720 upper=1.04720 effort=12.4 velocity=6.28
- added joint J_head_pitch: type revolute, parent Link_head_yaw, child Link_head_pitch, origin xyz=0 -0.0345999999999997 0.0484999999999999 rpy=0 0 0, axis 0 -1 0, limit lower=-0.7854 upper=0.7854 effort=26 velocity=109.8
- added joint J_head_yaw: type revolute, parent base_link, child Link_head_yaw, origin xyz=0.009 0 0.4064 rpy=0 0 0, axis 0 0 1, limit lower=-1.5708 upper=1.5708 effort=26 velocity=109.8
- added joint J_hip_l_pitch: type revolute, parent Link_hip_l_yaw, child Link_hip_l_pitch, origin xyz=0 -0.03675 -0.1055 rpy=0 0 0, axis 0 -1 0, limit lower=-0.78540 upper=1.83260 effort=396 velocity=19.16
- added joint J_hip_l_roll: type revolute, parent Link_waist_yaw, child Link_hip_l_roll, origin xyz=-0.0875 0.12 -0.069 rpy=0 0 0, axis 1 0 0, limit lower=-0.17453 upper=0.43633 effort=320 velocity=20.94
- added joint J_hip_l_yaw: type revolute, parent Link_hip_l_roll, child Link_hip_l_yaw, origin xyz=0.08225 0 -0.01 rpy=0 0 0, axis 0 0 1, limit lower=-0.69813 upper=0.69813 effort=160 velocity=19.63
- added joint J_hip_r_pitch: type revolute, parent Link_hip_r_yaw, child Link_hip_r_pitch, origin xyz=0 0.03675 -0.1055 rpy=0 0 0, axis 0 -1 0, limit lower=-0.78540 upper=1.83260 effort=396 velocity=19.16
- added joint J_hip_r_roll: type revolute, parent Link_waist_yaw, child Link_hip_r_roll, origin xyz=-0.0875 -0.12 -0.069 rpy=0 0 0, axis 1 0 0, limit lower=-0.17453 upper=0.43633 effort=320 velocity=20.94
- added joint J_hip_r_yaw: type revolute, parent Link_hip_r_roll, child Link_hip_r_yaw, origin xyz=0.08225 0 -0.01 rpy=0 0 0, axis 0 0 1, limit lower=-0.69813 upper=0.69813 effort=160 velocity=19.63
- added joint J_knee_l_pitch: type revolute, parent Link_hip_l_pitch, child Link_knee_l_pitch, origin xyz=0 0.01125 -0.4 rpy=0 0 0, axis 0 -1 0, limit lower=-2.35619 upper=0.08727 effort=396 velocity=19.16
- added joint J_knee_r_pitch: type revolute, parent Link_hip_r_pitch, child Link_knee_r_pitch, origin xyz=0 -0.01125 -0.4 rpy=0 0 0, axis 0 -1 0, limit lower=-2.35619 upper=0.08727 effort=396 velocity=19.16
- added joint J_waist_pitch: type revolute, parent base_link, child Link_waist_pitch, origin xyz=0 -0.0655 0 rpy=0 0 0, axis 0 -1 0, limit lower=-0.29671 upper=0.78540 effort=315 velocity=3.72
- added joint J_waist_roll: type revolute, parent Link_waist_pitch, child Link_waist_roll, origin xyz=-0.064 0.0655 0 rpy=0 0 0, axis 1 0 0, limit lower=-0.69813 upper=0.69813 effort=315 velocity=3.72
- added joint J_waist_yaw: type revolute, parent Link_waist_roll, child Link_waist_yaw, origin xyz=0.0675 0 -0.098 rpy=0 0 0, axis 0 0 1, limit lower=-0.78540 upper=0.78540 effort=121 velocity=5.92
